File: ABL Board - RP2040/ABL_RP2040.brd (EAGLE design)
At the start: 160 x 100 mm, 69 parts, among them P2 3.3V, Q1 MMBT4403, U1 RP2040, U2 W25Q128, U3 HX711, X1 CRYSTAL_TAXM12M4RLBDDT2T_3225, X2 LOADCELL 2, X3 LOADCELL 1, X4 LOADCELL 3, X5 INPUT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

Commit message: Pre review finalization
Parts:
- added U$1: (no value), FracktalWorks_Eagle_Library:FRACKTALLOGO
- moved C19 175.2 mm to (87.4, 25.4), turned to 270 degrees
- moved R16 173.9 mm to (80.3, 29.0)
- moved C18 172.7 mm to (97.5, 49.0)
- moved C17 168.9 mm to (92.7, 50.8)
- moved Z_OUT 168.9 mm to (77.5, 31.8), turned to 270 degrees
- moved X6 167.3 mm to (81.0, 23.9)
- moved C23 164.8 mm to (90.2, 25.7), turned to 270 degrees
- moved C16 161.7 mm to (93.5, 62.5), turned to 180 degrees
- moved C26 160.4 mm to (89.2, 46.5), turned to 270 degrees
- moved C22 160.1 mm to (91.7, 32.5), turned to 90 degrees
- moved X1 159.8 mm to (69.3, 33.0)
- moved P2 159.1 mm to (90.2, 56.1), turned to 180 degrees
- moved R2 158.9 mm to (77.2, 50.8), turned to 90 degrees
- moved R3 158.1 mm to (69.8, 36.6), turned to 90 degrees
- moved C20 154.9 mm to (96.0, 38.4), turned to 270 degrees
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Routing:
- net GND: track 0.00 -> 360.0 mm, vias 0 -> 37
- net +5V: track 0.00 -> 136.3 mm, vias 0 -> 2
- net +3.3V: track 0.00 -> 124.5 mm, vias 0 -> 3
- net A-: track 0.00 -> 81.4 mm, vias 0 -> 1
- net AVDD: track 0.00 -> 79.9 mm, vias 0 -> 2
- net A+: track 0.00 -> 76.4 mm, vias 0 -> 1
- net RESET: track 0.00 -> 61.5 mm, vias 0 -> 2
- net SCK: track 0.00 -> 56.2 mm, vias 0 -> 2
- net DAT: track 0.00 -> 55.0 mm, vias 0 -> 2
- net Z_OUT: track 0.00 -> 45.2 mm
- net ABL_LED: track 0.00 -> 42.0 mm, vias 0 -> 2
- net USB1_P: track 0.00 -> 41.1 mm
- net USB1_N: track 0.00 -> 39.2 mm, vias 0 -> 2
- net QSPI_SS: track 0.00 -> 29.1 mm
- net +1.1V: track 0.00 -> 28.0 mm, vias 0 -> 3
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- added copper zone on layer 1, net GND
- added copper zone on layer 16, net GND
Other:
- board size 160 x 100 mm -> 62.2 x 63.5 mm
- board text added: "+"
- board text added: "+3.3V"
- board text added: "+5V"
- board text added: "-"
- board text added: "ABL Board V3"
- board text added: "ABL LED"
- board text added: "Design by Nishant Bilurkar"
- board text added: "GND"
- board text added: "LOADCELL 1"
- board text added: "LOADCELL 2"
- board text added: "LOADCELL 3"
- board text added: "POWER"
- board text added: "USB_N"
- board text added: "USB_P"
- board text added: "Z_OUT"
