File: Multi Extruder Board/Stepper motor board.brd (EAGLE design)
At the start: 161 x 109.5 mm, 156 parts, among them P1 TPS54202_BUCKCONV, P2 3.3V, U1 RP2040IC57_RP2040-L, U2 W25Q128JVSIQSOIC_128JVSIQ_WIN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, U3 SN65HVD, X1 CRYSTAL_TAXM12M4RLBDDT2T_3225, X18 JST-XH-02-PIN-LONG-PAD, X19 JST-XH-02-PIN-LONG-PAD, X2 JST-XH-04-PIN-LONG-PAD, X20 JST-XH-02-PIN-LONG-PAD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

Commit message: Logo, BOM, Centroids, Gerber files changes
Parts:
- renumbered U$1 to U$3
Other:
- board size 161 x 109.5 mm -> 120 x 74.5 mm
- board text removed: "BOOT"
- board text removed: "BUCK CONVERTOR"
- board text removed: "BUTTONS 0"
- board text removed: "BUTTONS 1"
- board text removed: "BUTTONS 2"
- board text removed: "BUTTONS 3"
- board text removed: "CANBUS"
- board text removed: "CRYSTAL"
- board text removed: "EXTRUDER 0"
- board text removed: "EXTRUDER 1"
- board text removed: "EXTRUDER 2"
- board text removed: "EXTRUDER 3"
- board text removed: "EXTRUDER PINS"
- board text removed: "FLASH"
- board text removed: "LDO"
- board text removed: "USB"
Changed lines of the file:
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@@
 <board>
 <plain>
-<wire x1="0" y1="-1" x2="23" y2="-1" width="0" layer="20"/>
-<wire x1="128" y1="-1" x2="160" y2="-1" width="0" layer="20"/>
-<wire x1="160" y1="-1" x2="161" y2="108.5" width="0" layer="20"/>
-<wire x1="161" y1="108.5" x2="1" y2="108.5" width="0" layer="20"/>
-<wire x1="1" y1="108.5" x2="0" y2="-1" width="0" layer="20"/>
-<wire x1="-111.887" y1="102.87" x2="-111.887" y2="91.44" width="0.1524" layer="48"/>
-<wire x1="-111.887" y1="91.44" x2="-97.028" y2="91.44" width="0.1524" layer="48"/>
-<wire x1="-97.028" y1="91.44" x2="-97.028" y2="102.87" width="0.1524" layer="48"/>
-<wire x1="-97.028" y1="102.87" x2="-111.887" y2="102.87" width="0.1524" layer="48"/>
-<text x="-110.617" y="100.584" size="1.27" layer="48">CRYSTAL</text>
-<wire x1="-78.486" y1="117.475" x2="-78.486" y2="92.075" width="0.1524" layer="48"/>
-<wire x1="-78.486" y1="92.075" x2="-33.147" y2="92.075" width="0.1524" layer="48"/>
-<wire x1="-33.147" y1="92.075" x2="-33.147" y2="117.475" width="0.1524" layer="48"/>
-<wire x1="-33.147" y1="117.475" x2="-78.486" y2="117.475" width="0.1524" layer="48"/>
-<text x="-76.708" y="113.792" size="1.778" layer="48">BUCK CONVERTOR</text>
-<wire x1="-124.46" y1="60.96" x2="-124.46" y2="35.814" width="0.1524" layer="48"/>
-<wire x1="-124.46" y1="35.814" x2="-97.028" y2="35.814" width="0.1524" layer="48"/>
-<wire x1="-97.028" y1="35.814" x2="-97.028" y2="60.96" width="0.1524" layer="48"/>
-<wire x1="-97.028" y1="60.96" x2="-124.46" y2="60.96" width="0.1524" layer="48"/>
-<text x="-122.936" y="57.15" size="1.778" layer="48">CANBUS</text>
-<wire x1="-160.02" y1="-1.016" x2="-160.02" y2="-50.8" width="0.1524" layer="48"/>
-<wire x1="-160.02" y1="-50.8" x2="-114.554" y2="-50.8" width="0.1524" layer="48"/>
-<wire x1="-114.554" y1="-50.8" x2="-114.554" y2="-1.016" width="0.1524" layer="48"/>
-<wire x1="-114.554" y1="-1.016" x2="-160.02" y2="-1.016" width="0.1524" layer="48"/>
-<text x="-155.702" y="-4.318" size="1.778" layer="48">USB</text>
-<wire x1="-53.467" y1="49.149" x2="-53.467" y2="35.56" width="0.1524" layer="48"/>
-<wire x1="-53.467" y1="35.56" x2="-14.605" y2="35.56" width="0.1524" layer="48"/>
-<wire x1="-14.605" y1="35.56" x2="-14.605" y2="49.149" width="0.1524" layer="48"/>
-<wire x1="-14.605" y1="49.149" x2="-53.467" y2="49.149" width="0.1524" layer="48"/>
-<text x="-25.019" y="38.608" size="1.778" layer="48">FLASH</text>
-<wire x1="-10" y1="-18" x2="-10" y2="-51" width="0.1524" layer="48"/>
-<wire x1="-10" y1="-51" x2="37" y2="-51" width="0.1524" layer="48"/>
-<wire x1="37" y1="-51" x2="37" y2="-18" width="0.1524" layer="48"/>
-<wire x1="37" y1="-18" x2="-10" y2="-18" width="0.1524" layer="48"/>
-<text x="-7" y="-23" size="1.778" layer="48">EXTRUDER 0</text>
-<wire x1="42" y1="-18" x2="42" y2="-51" width="0.1524" layer="48"/>
-<wire x1="42" y1="-51" x2="81" y2="-51" width="0.1524" layer="48"/>
-<wire x1="81" y1="-51" x2="81" y2="-18" width="0.1524" layer="48"/>
-<wire x1="81" y1="-18" x2="42" y2="-18" width="0.1524" layer="48"/>
-<text x="45" y="-23" size="1.778" layer="48">EXTRUDER 1</text>
-<wire x1="90" y1="-18" x2="90" y2="-51" width="0.1524" layer="48"/>
-<wire x1="90" y1="-51" x2="127" y2="-51" width="0.1524" layer="48"/>
-<wire x1="127" y1="-51" x2="127" y2="-18" width="0.1524" layer="48"/>
-<wire x1="127" y1="-18" x2="90" y2="-18" width="0.1524" layer="48"/>
-<text x="94" y="-23" size="1.778" layer="48">EXTRUDER 2</text>
-<wire x1="143" y1="-18" x2="143" y2="-51" width="0.1524" layer="48"/>
-<wire x1="143" y1="-51" x2="177" y2="-51" width="0.1524" layer="48"/>
-<wire x1="177" y1="-51" x2="177" y2="-18" width="0.1524" layer="48"/>
-<wire x1="177" y1="-18" x2="143" y2="-18" width="0.1524" layer="48"/>
-<text x="146" y="-23" size="1.778" layer="48">EXTRUDER 3</text>
-<wire x1="-113" y1="88" x2="-113" y2="71" width="0.1524" layer="48"/>
-<wire x1="-113" y1="71" x2="-93" y2="71" width="0.1524" layer="48"/>
-<wire x1="-93" y1="71" x2="-93" y2="88" width="0.1524" layer="48"/>
-<wire x1="-93" y1="88" x2="-113" y2="88" width="0.1524" layer="48"/>
-<text x="-110" y="84" size="1.778" layer="48">LDO</text>
-<wire x1="-92" y1="58" x2="-92" y2="-5" width="0.1524" layer="48"/>
-<wire x1="-92" y1="-5" x2="-64" y2="-5" width="0.1524" layer="48"/>
-<wire x1="-64" y1="-5" x2="-64" y2="58" width="0.1524" layer="48"/>
-<wire x1="-64" y1="58" x2="-92" y2="58" width="0.1524" layer="48"/>
-<text x="-88" y="54" size="1.778" layer="48">EXTRUDER PINS</text>
-<wire x1="-106" y1="-39" x2="-106" y2="-83" width="0.1524" layer="48"/>
-<wire x1="-106" y1="-83" x2="-42" y2="-83" width="0.1524" layer="48"/>
-<wire x1="-42" y1="-83" x2="-42" y2="-39" width="0.1524" layer="48"/>
-<wire x1="-42" y1="-39" x2="-106" y2="-39" width="0.1524" layer="48"/>
-<text x="-97" y="-45" size="1.778" layer="48">BUTTONS 0</text>
-<wire x1="-104" y1="-106" x2="-104" y2="-151" width="0.1524" layer="48"/>
-<wire x1="-104" y1="-151" x2="-46" y2="-151" width="0.1524" layer="48"/>
-<wire x1="-46" y1="-151" x2="-46" y2="-106" width="0.1524" layer="48"/>
-<wire x1="-46" y1="-106" x2="-104" y2="-106" width="0.1524" layer="48"/>
-<text x="-96" y="-112" size="1.778" layer="48">BUTTONS 1</text>
-<wire x1="-104" y1="-159" x2="-104" y2="-194" width="0.1524" layer="48"/>
-<wire x1="-104" y1="-194" x2="-50" y2="-194" width="0.1524" layer="48"/>
-<wire x1="-50" y1="-194" x2="-50" y2="-159" width="0.1524" layer="48"/>
-<wire x1="-50" y1="-159" x2="-104" y2="-159" width="0.1524" layer="48"/>
-<text x="-66" y="-172" size="1.778" layer="48">BUTTONS 2</text>
-<wire x1="-99" y1="-207" x2="-99" y2="-239" width="0.1524" layer="48"/>
-<wire x1="-99" y1="-239" x2="-43" y2="-239" width="0.1524" layer="48"/>
-<wire x1="-43" y1="-239" x2="-43" y2="-207" width="0.1524" layer="48"/>
-<wire x1="-43" y1="-207" x2="-99" y2="-207" width="0.1524" layer="48"/>
-<text x="-98" y="-218" size="1.778" layer="48">BUTTONS 3</text>
-<wire x1="-100" y1="-244" x2="-100" y2="-284" width="0.1524" layer="48"/>
-<wire x1="-100" y1="-284" x2="-40" y2="-284" width="0.1524" layer="48"/>
-<wire x1="-40" y1="-284" x2="-40" y2="-244" width="0.1524" layer="48"/>
-<wire x1="-40" y1="-244" x2="-100" y2="-244" width="0.1524" layer="48"/>
-<text x="-93" y="-250" size="1.778" layer="48">BOOT</text>
 <wire x1="18" y1="73.5" x2="18" y2="-1" width="0.1524" layer="51"/>
 <wire x1="18" y1="-1" x2="138" y2="-1" width="0.1524" layer="51"/>
@@
 <element name="FS1" library="SparkFun-Connectors" library_urn="urn:adsk.eagle:library:513" package="PAD.03X.04" package3d_urn="urn:adsk.eagle:package:38287/1" value="TEST-POINT3X4" x="136" y="33.5" smashed="yes"/>
 <element name="FS3" library="SparkFun-Connectors" library_urn="urn:adsk.eagle:library:513" package="PAD.03X.04" package3d_urn="urn:adsk.eagle:package:38287/1" value="TEST-POINT3X4" x="136" y="28.5" smashed="yes"/>
-<element name="U$1" library="FracktalWorks_Eagle_Library" package="FWLOGO_SMALL" value="" x="40" y="32.5" smashed="yes"/>
 <element name="U$2" library="FracktalWorks_Eagle_Library" package="MAKEININDIA" value="" x="41.2088" y="47.079" smashed="yes"/>
+<element name="U$3" library="FracktalWorks_Eagle_Library" package="FWLOGO_SMALL" value="" x="40" y="32.5" smashed="yes"/>
 </elements>
 <signals>
